Commit message: 28.07

File: mir_description/urdf/include/mir_v1.urdf.xacro (robot description, xacro)
@@ -1,6 +1,6 @@
 <?xml version="1.0"?>
 <robot xmlns:xacro="http://ros.org/wiki/xacro">
-  <xacro:arg name="mir_type" default="mir_100" />      <!-- The MiR variant. Can be "mir_100" or "mir_250" for now.-->
-  <xacro:property name="mir_type" value="$(arg mir_type)" />  <!-- necessary because args cannot be accessed inside ${} expressions -->
+  <xacro:arg name="mir_type" default="mir_100" /> <!-- The MiR variant. Can be "mir_100" or "mir_250" for now.-->
+  <xacro:property name="mir_type" value="$(arg mir_type)" /> <!-- necessary because args cannot be accessed inside ${} expressions -->
   <xacro:include filename="$(find mir_description)/urdf/include/common_properties.urdf.xacro" />
   <xacro:include filename="$(find mir_description)/urdf/include/imu.gazebo.urdf.xacro" />
@@ -8,4 +8,5 @@
   <xacro:include filename="$(find mir_description)/urdf/include/mir.transmission.xacro" />
   <xacro:include filename="$(find mir_description)/urdf/include/sick_s300.urdf.xacro" />
+  <xacro:include filename="$(find mir_description)/urdf/include/intel_d435.urdf.xacro" />
   <xacro:property name="deg_to_rad" value="0.017453293" />
   <!-- The inertia for the MiR platform is intentionally chosen to be smaller than
@@ -42,9 +43,9 @@
   <xacro:property name="mir_front_caster_wheel_base_dx" value="0.3037" />
   <xacro:if value="${mir_type == 'mir_100'}">
-    <xacro:property name="mir_back_caster_wheel_base_dx"  value="0.3078" />
+    <xacro:property name="mir_back_caster_wheel_base_dx" value="0.3078" />
     <xacro:property name="mir_caster_wheel_base_dy" value="0.203" />
   </xacro:if>
   <xacro:if value="${mir_type == 'mir_250'}">
-    <xacro:property name="mir_back_caster_wheel_base_dx"  value="0.296" />
+    <xacro:property name="mir_back_caster_wheel_base_dx" value="0.296" />
     <xacro:property name="mir_caster_wheel_base_dy" value="0.188" />
   </xacro:if>
@@ -97,5 +98,5 @@
       <child link="${prefix}${locationprefix}_caster_rotation_link" />
       <axis xyz="0 0 1" />
-      <dynamics damping="0.01" friction="0.0"/>
+      <dynamics damping="0.01" friction="0.0" />
     </joint>
     <link name="${prefix}${locationprefix}_caster_rotation_link">
@@ -104,11 +105,5 @@
         <origin xyz="0 0 -0.042500000044" rpy="${24 * deg_to_rad} 0 ${0.5 * pi} " />
         <mass value="0.3097539019" />
-        <inertia
-          ixx="0.0005844517978"
-          ixy="0"
-          ixz="0"
-          iyy="0.00052872551237"
-          iyz="0"
-          izz="0.00017923555074" />
+        <inertia ixx="0.0005844517978" ixy="0" ixz="0" iyy="0.00052872551237" iyz="0" izz="0.00017923555074" />
       </inertial>
       <visual>
@@ -210,5 +205,5 @@
       <parent link="${prefix}base_link" />
       <child link="${prefix}imu_link" />
-      <origin xyz="0.0 0.0 0.25" rpy="0 0 0" />  <!-- same as real MiR -->
+      <origin xyz="0.0 0.0 0.25" rpy="0 0 0" /> <!-- same as real MiR -->
     </joint>
     <link name="${prefix}imu_link" />
@@ -223,4 +218,8 @@
     </joint>
     <link name="${prefix}imu_frame" />
+    <!-- Intel Realsense -->
+    <xacro:sensor_intel_d435i prefix="realsense_rgbd" parent="${prefix}base_link" prefix_topic="realsense">
+      <origin xyz="0.47 0 0.28" rpy="0 0 0" />
+    </xacro:sensor_intel_d435i>
     <!-- Laser scanners -->
     <joint name="${prefix}base_link_to_front_laser_joint" type="fixed">
@@ -237,23 +236,25 @@
     <xacro:sick_s300 prefix="${prefix}" link="back_laser_link" topic="b_scan" />
     <!-- Ultrasound sensors -->
-    <joint name="${prefix}us_1_joint" type="fixed">   <!-- right ultrasound -->
+    <joint name="${prefix}us_1_joint" type="fixed">
+      <!-- right ultrasound -->
       <parent link="${prefix}base_link" />
       <child link="${prefix}us_1_frame" />
-      <origin xyz="0.45 -0.12 0.16 " rpy="0 0 0" />  <!-- from visually matching to the mesh of the MiR -->
+      <origin xyz="0.45 -0.12 0.16 " rpy="0 0 0" /> <!-- from visually matching to the mesh of the MiR -->
     </joint>
     <link name="${prefix}us_1_frame" />
-    <joint name="${prefix}us_2_joint" type="fixed">   <!-- left ultrasound -->
+    <joint name="${prefix}us_2_joint" type="fixed">
+      <!-- left ultrasound -->
       <parent link="${prefix}base_link" />
       <child link="${prefix}us_2_frame" />
-      <origin xyz="0.45 0.12 0.16 " rpy="0 0 0" />  <!-- from visually matching to the mesh of the MiR -->
+      <origin xyz="0.45 0.12 0.16 " rpy="0 0 0" /> <!-- from visually matching to the mesh of the MiR -->
     </joint>
     <link name="${prefix}us_2_frame" />
     <!-- wheels -->
-    <xacro:actuated_wheel prefix="${prefix}" locationprefix="left" locationright="-1"/>
-    <xacro:actuated_wheel prefix="${prefix}" locationprefix="right" locationright="1"/>
-    <xacro:caster_wheel prefix="${prefix}" locationprefix="fl" locationright="-1" wheel_base_dx="${mir_front_caster_wheel_base_dx + mir_act_wheel_dx}"/>
-    <xacro:caster_wheel prefix="${prefix}" locationprefix="fr" locationright="1" wheel_base_dx="${mir_front_caster_wheel_base_dx + mir_act_wheel_dx}"/>
-    <xacro:caster_wheel prefix="${prefix}" locationprefix="bl" locationright="-1" wheel_base_dx="${-mir_back_caster_wheel_base_dx + mir_act_wheel_dx}"/>
-    <xacro:caster_wheel prefix="${prefix}" locationprefix="br" locationright="1" wheel_base_dx="${-mir_back_caster_wheel_base_dx + mir_act_wheel_dx}"/>
+    <xacro:actuated_wheel prefix="${prefix}" locationprefix="left" locationright="-1" />
+    <xacro:actuated_wheel prefix="${prefix}" locationprefix="right" locationright="1" />
+    <xacro:caster_wheel prefix="${prefix}" locationprefix="fl" locationright="-1" wheel_base_dx="${mir_front_caster_wheel_base_dx + mir_act_wheel_dx}" />
+    <xacro:caster_wheel prefix="${prefix}" locationprefix="fr" locationright="1" wheel_base_dx="${mir_front_caster_wheel_base_dx + mir_act_wheel_dx}" />
+    <xacro:caster_wheel prefix="${prefix}" locationprefix="bl" locationright="-1" wheel_base_dx="${-mir_back_caster_wheel_base_dx + mir_act_wheel_dx}" />
+    <xacro:caster_wheel prefix="${prefix}" locationprefix="br" locationright="1" wheel_base_dx="${-mir_back_caster_wheel_base_dx + mir_act_wheel_dx}" />
     <joint name="${prefix}base_link_surface_joint" type="fixed">
       <origin xyz="${mir_act_wheel_dx} 0 0.352" rpy="0 0 0" />
@@ -262,8 +263,8 @@
       <axis xyz="0 0 1" />
     </joint>
-    <link name="${prefix}surface"/>
-    <xacro:mir_wheel_transmissions prefix="${prefix}"/>
+    <link name="${prefix}surface" />
+    <xacro:mir_wheel_transmissions prefix="${prefix}" />
     <!-- set the gazebo friction parameters for the wheels -->
-    <xacro:set_all_wheel_frictions prefix="${prefix}"/>
+    <xacro:set_all_wheel_frictions prefix="${prefix}" />
     <xacro:p3d_base_controller prefix="${prefix}" />
   </xacro:macro>
